File: circuit/eagle/USBCharger.sch (EAGLE design)
At the start: 39 parts, among them IC1 ATMEGA168-20P, IC2 7400N, IC3 74HCT574N, IC4 74HCT574N, IC6 74LS30N, IC7 74LS00N, IC8 74LS00N, IC9 74HCT574N, X1 PN61729-S

Commit message: updated circuit files
Parts:
- added R8, R9: 10k, resistor:R-EU_0204/7
Connections:
- net GND: now also R8.1, R9.1
- net PB0_EE_EN: now also R8.2
- net PD3_EE_RW: now also R9.2
Other:
- note added: "* added two pulldown resistors to keep safe eeprom during MCU cold start & flashing"
Changed lines of the file:
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@@
 <part name="P+6" library="supply1" deviceset="+5V" device=""/>
 <part name="GND8" library="supply1" deviceset="GND" device=""/>
+<part name="R8" library="resistor" deviceset="R-EU_" device="0204/7" value="10k"/>
+<part name="R9" library="resistor" deviceset="R-EU_" device="0204/7" value="10k"/>
+<part name="GND9" library="supply1" deviceset="GND" device=""/>
 </parts>
 <sheets>
@@
 <wire x1="129.54" y1="-22.86" x2="129.54" y2="-50.8" width="0.1524" layer="94"/>
 <text x="124.46" y="-48.26" size="1.778" layer="94" rot="R270">1FF4-1FFB Active LOW Trigger</text>
+<text x="-17.78" y="-20.32" size="1.778" layer="91">* added two pulldown resistors
+to keep safe eeprom during
+MCU cold start &amp; flashing</text>
 </plain>
 <instances>
@@
 <instance part="P+6" gate="1" x="177.8" y="15.24"/>
 <instance part="GND8" gate="1" x="190.5" y="-45.72"/>
+<instance part="R8" gate="G$1" x="-22.86" y="-10.16" rot="R90"/>
+<instance part="R9" gate="G$1" x="-30.48" y="-5.08" rot="R90"/>
+<instance part="GND9" gate="1" x="-30.48" y="-20.32"/>
 </instances>
 <busses>
@@
 <junction x="-22.86" y="7.62"/>
 <wire x1="-22.86" y1="35.56" x2="-22.86" y2="7.62" width="0.1524" layer="91"/>
+<pinref part="R8" gate="G$1" pin="2"/>
+<junction x="-22.86" y="-5.08"/>
 </segment>
 <segment>
@@
 <junction x="190.5" y="-43.18"/>
 </segment>
+<segment>
+<pinref part="R9" gate="G$1" pin="1"/>
+<pinref part="GND9" gate="1" pin="GND"/>
+<wire x1="-30.48" y1="-10.16" x2="-30.48" y2="-17.78" width="0.1524" layer="91"/>
+<pinref part="R8" gate="G$1" pin="1"/>
+<wire x1="-22.86" y1="-15.24" x2="-22.86" y2="-17.78" width="0.1524" layer="91"/>
+<wire x1="-22.86" y1="-17.78" x2="-30.48" y2="-17.78" width="0.1524" layer="91"/>
+<junction x="-30.48" y="-17.78"/>
+</segment>
 </net>
 <net name="+5V" class="0">
@@
 <label x="-33.02" y="22.86" size="1.778" layer="95"/>
 <pinref part="IC2" gate="A" pin="I0"/>
-<wire x1="-20.32" y1="22.86" x2="-33.02" y2="22.86" width="0.1524" layer="91"/>
+<wire x1="-20.32" y1="22.86" x2="-30.48" y2="22.86" width="0.1524" layer="91"/>
+<wire x1="-30.48" y1="22.86" x2="-33.02" y2="22.86" width="0.1524" layer="91"/>
 <wire x1="-20.32" y1="27.94" x2="-17.78" y2="27.94" width="0.1524" layer="91"/>
 <wire x1="-20.32" y1="27.94" x2="-20.32" y2="22.86" width="0.1524" layer="91"/>
@@
 <wire x1="-17.78" y1="0" x2="-20.32" y2="0" width="0.1524" layer="91"/>
 <wire x1="-20.32" y1="0" x2="-20.32" y2="22.86" width="0.1524" layer="91"/>
+<pinref part="R9" gate="G$1" pin="2"/>
+<wire x1="-30.48" y1="0" x2="-30.48" y2="22.86" width="0.1524" layer="91"/>
+<junction x="-30.48" y="22.86"/>
 </segment>
 <segment>
@@
 </schematic>
 </drawing>
+<compatibility>
+<note version="6.3" minversion="6.2.2" severity="warning">
+Since Version 6.2.2 text objects can contain more than one line,
+which will not be processed correctly with this version.
+</note>
+</compatibility>
 </eagle>
